Commit message: gazebo references

File: description/robot_core.xacro (robot description, xacro)
@@ -40,4 +40,7 @@
         </xacro:inertial_box>
     </link>
+    <gazebo reference="chassis">
+        <material>Gazebo/White</material>
+    </gazebo>
     <!-- LEFT WHEEL-->
     <joint name="left_wheel_joint" type="continuous">
@@ -63,4 +66,7 @@
         </xacro:inertial_cylinder>
     </link>
+    <gazebo reference="left_wheel">
+        <material>Gazebo/Black</material>
+    </gazebo>
     <!-- RIGHT WHEEL-->
     <joint name="right_wheel_joint" type="continuous">
@@ -86,4 +92,7 @@
         </xacro:inertial_cylinder>
     </link>
+    <gazebo reference="right_wheel">
+        <material>Gazebo/Black</material>
+    </gazebo>
     <!-- CASTER WHEEL-->
     <joint name="caster_wheel_joint" type="fixed">
@@ -108,3 +117,8 @@
         </xacro:inertial_sphere>
     </link>
+    <gazebo reference="caster_wheel">
+        <material>Gazebo/Black</material>
+        <nul1 value="0.001"/>
+        <nul2 value="0.001"/>
+    </gazebo>
 </robot>

Commit message: robot update

File: description/robot_core.xacro (robot description, xacro)
@@ -13,4 +13,7 @@
     <material name="orange">
         <color rgba="1 0.3 0.1 1"/>
+    </material>
+    <material name="red">
+        <color rgba="1 0 0 1"/>
     </material>
     <link name="base_link">
