Commit message: Colors update

File: description/camera.xacro (robot description, xacro)
@@ -11,5 +11,5 @@
                 <box size="0.010 0.03 0.03"/>
             </geometry>
-            <material name="red"/>
+            <material name="black"/>
         </visual>
     </link>
@@ -21,5 +21,5 @@
     <link name="camera_link_optical"> </link>
     <gazebo reference="camera_link">
-        <material>Gazebo/Red</material>
+        <material>Gazebo/Black</material>
         <sensor name="camera" type="camera">
             <pose> 0 0 0 0 0 0</pose>
